File: Robot-Simple-PCB/Robot-Simple-PCB.kicad_pcb (KiCad board)
At the start: 2 copper layers, 91 parts, among them J1 Main Power In, J10 PiicoDev, J11 MotA, J12 MotB, J13 Mot3, J14 Ext_PWR_Sw, J15 PSU_in, J16 PSU_out, J17 WS2812_Out, J18 Prog_Header, J19 Breakout_Header, J2 Servo1, J20 UART_Conn, J3 Servo1, J4 Servo2, J5 Servo2, J6 Servo3, J7 Servo4, J8 Plug and pair, Q3 Q_PMOS_GDS, Q4 Q_PMOS_GDS, SW1 Onboard_PWR_Sw, SW2 User_Button, U1 74LVC2G34GW, U2 DRV8871DDA, U3 DRV8871DDA, U4 DRV8871DDA, U5 AMS1117-3.3, U6 TPS54302, U7 ESP32-S3-WROOM-1, U8 74LVC2G34GW

Commit message: Schematic complete, started routing
Parts:
- added D8: D_Schottky, Diode_SMD:D_SOD-123, F.Cu at (-17.9, 22.4)
- added D9: D_Schottky, Diode_SMD:D_SOD-123, F.Cu at (-17.9, 25.8)
- added P1: USB_C_Plug_USB2.0, Connector_USB:USB_C_Receptacle_GCT_USB4125-xx-x_6P_TopMnt_Horizontal, F.Cu at (-21.5, 6.63)
- added R27: 5.1k, Resistor_SMD:R_0402_1005Metric_Pad0.72x0.64mm_HandSolder, F.Cu at (-13.4, 21.8)
- added R28: 5.1k, Resistor_SMD:R_0402_1005Metric_Pad0.72x0.64mm_HandSolder, F.Cu at (-13.4, 23.8)
- moved J13 213.1 mm to (245.4, 50.8)
- moved SW1 184.1 mm to (-29.1, 49.4)
- moved U4 167.6 mm to (226.4, 22.2)
- moved U3 156.9 mm to (225.7, 36.2)
- moved J8 147.3 mm to (99.1, -35.6)
- moved U2 147.2 mm to (224.2, 50.8)
- moved C8 138.1 mm to (112.2, -15.2)
- moved D11 135.0 mm to (174.5, -7.62)
- moved J2 134.9 mm to (215.9, 109.2)
- moved J3 134.9 mm to (220.6, 109.2)
- moved J6 134.9 mm to (234.5, 109.2)
- moved J7 134.9 mm to (239.2, 109.2)
- moved J4 134.9 mm to (225.2, 109.2)
- moved J5 134.9 mm to (229.8, 109.2)
- moved D7 134.3 mm to (172.7, -12.7)
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Connections:
- D12 pad 1: +5VP -> +5V
- D3 pad 1: +5VP -> +5V
- JP1 pad 2: unconnected-(JP1-B-Pad2) -> Net-(D8-A)

Commit message: Yuuuuh
Parts:
- removed JP3: Rev_Volt_out, Jumper:SolderJumper-2_P1.3mm_Open_RoundedPad1.0x1.5mm
- removed P1: USB_C_Plug_USB2.0, Connector_USB:USB_C_Receptacle_GCT_USB4125-xx-x_6P_TopMnt_Horizontal
- added C9: 10u, Capacitor_SMD:C_1206_3216Metric, F.Cu at (68.8, 37.9)
- added J9: USB_C_Receptacle_USB2.0_16P, Connector_USB:USB_C_Receptacle_HCTL_HC-TYPE-C-16P-01A, F.Cu at (113.1, 61.8)
- C1, C2, C5, C6: footprint Capacitor_SMD:C_0402_1005Metric -> Capacitor_SMD:C_1206_3216Metric
- C3, C4: footprint Capacitor_SMD:C_0402_1005Metric -> Capacitor_SMD:C_0603_1608Metric
- R21, R22: value R -> 10k
- moved J19 239.0 mm to (43.8, 63.5), turned to 90 degrees
- moved J11 167.3 mm to (76.6, 23.5)
- moved J20 160.9 mm to (33.8, 46.1)
- moved J12 159.2 mm to (86.7, 23.6)
- moved R25 154.3 mm to (113.0, 39.0), turned to 90 degrees
- moved R8 153.0 mm to (83.5, 39.6), turned to 90 degrees
- moved J13 151.1 mm to (96.8, 23.6)
- moved R24 148.6 mm to (111.0, 38.8), turned to 90 degrees
- moved J5 148.2 mm to (107.5, 25.7), turned to 180 degrees
- moved U4 148.0 mm to (78.8, 33.3), turned to 90 degrees
- moved U8 146.7 mm to (113.8, 42.5), turned to 90 degrees
- moved R7 144.5 mm to (80.8, 39.5), turned to -90 degrees
- moved J6 144.3 mm to (116.8, 25.7), turned to 180 degrees
- moved J7 143.0 mm to (116.8, 35.2), turned to 180 degrees
- moved R10 141.7 mm to (93.6, 39.6), turned to 90 degrees
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Connections:
- C2 pad 1: Net-(JP2-B) -> Net-(J15-Pin_2)
- C3 pad 1: Net-(JP2-B) -> Net-(J15-Pin_2)
- C5 pad 1: +5VP -> Net-(JP1-A)
- C6 pad 1: +5VP -> Net-(JP1-A)
- D8 pad 1: Net-(D8-K) -> +5V
- D8 pad 2: Net-(D8-A) -> +5VP
- D9 pad 1: Net-(D8-K) -> +5V
- D9 pad 2: +5V -> VBUS
- J10 pad 2: +3.3V -> +3V3
- J15 pad 2: VBAT -> Net-(J15-Pin_2)
- J16 pad 2: Net-(D8-K) -> +5V
- J19 pad 4: /BKT_IO13 -> /BKT_IO40
- J19 pad 5: /BKT_IO14 -> /BKT_IO41
- J19 pad 6: /BKT_IO15 -> /BKT_IO42
- J19 pad 7: /BKT_IO16 -> /BKT_IO2
- J19 pad 9: /BKT_IO21 -> /BKT_IO1
- J20 pad 4: +3.3V -> +3V3
- JP1 pad 1: +5VP -> Net-(JP1-A)
- JP1 pad 2: Net-(D8-A) -> +5VP
- JP2 pad 2: Net-(JP2-B) -> Net-(J15-Pin_2)
- L1 pad 2: +5VP -> Net-(JP1-A)
- Q4 pad 2: Net-(JP3-A) -> VBAT
- R1 pad 1: +3.3V -> +3V3
- R15 pad 1: Net-(JP2-B) -> Net-(J15-Pin_2)
- R17 pad 1: +5VP -> Net-(JP1-A)
- R2 pad 1: +3.3V -> +3V3
- R5 pad 1: Net-(JP3-A) -> VBAT
- TP3 pad 1: Net-(JP3-A) -> VBAT
- TP5 pad 1: +5VP -> Net-(JP1-A)
- U2 pad 6: Net-(J13-Pin_1) -> Net-(J13-Pin_2)
- U2 pad 8: Net-(J13-Pin_2) -> Net-(J13-Pin_1)
- U3 pad 6: Net-(J12-Pin_1) -> Net-(J12-Pin_2)
- U3 pad 8: Net-(J12-Pin_2) -> Net-(J12-Pin_1)
- U4 pad 6: Net-(J11-Pin_1) -> Net-(J11-Pin_2)
- U4 pad 8: Net-(J11-Pin_2) -> Net-(J11-Pin_1)
- U5 pad 3: Net-(D8-K) -> +5V
- U6 pad 3: Net-(JP2-B) -> Net-(J15-Pin_2)
- U7 pad 10: /HB_LED -> /Servo_Sig_4
- U7 pad 11: /USER_WS2812 -> /HB_LED
- U7 pad 12: /UART0_RXD -> /Servo_Sig_3
- U7 pad 17: /UART0_TXD -> /Servo_Sig_2
- U7 pad 18: /PAIR_LED -> /Servo_Sig_1
- U7 pad 19: /UART1_RXD -> /Mot3_A
- U7 pad 20: /UART1_TXD -> /Mot3_B
- U7 pad 21: /BKT_IO13 -> /Mot2_A
- U7 pad 22: /BKT_IO14 -> /Mot2_B
- U7 pad 23: /BKT_IO21 -> /Mot1_A
- U7 pad 24: /Mot3_A -> /Mot1_B
- U7 pad 25: /Mot3_B -> /UART1_TXD
- U7 pad 31: /Mot1_A -> /UART1_RXD
- U7 pad 32: /Mot1_B -> /USER_WS2812
- U7 pad 33: /Mot2_A -> /BKT_IO40
- U7 pad 34: /Mot2_B -> /BKT_IO41
- U7 pad 35: /USER_BUTTON -> /BKT_IO42
- U7 pad 38: /Servo_Sig_2 -> /BKT_IO2
- U7 pad 39: /Servo_Sig_1 -> /BKT_IO1
- U7 pad 4: /Servo_Sig_3 -> /UART0_RXD
- U7 pad 5: /Servo_Sig_4 -> /UART0_TXD
- U7 pad 6: /I2C0_SDA -> /PAIR_LED
- U7 pad 7: /I2C0_SCL -> /USER_BUTTON
- U7 pad 8: /BKT_IO15 -> /I2C0_SDA
- U7 pad 9: /BKT_IO16 -> /I2C0_SCL
Routing:
- net +5VP: track 0.00 -> 142.3 mm, vias 0 -> 4
- net +3V3: track 0.00 -> 139.6 mm, vias 0 -> 5
- net +5V: track 0.00 -> 103.3 mm, vias 0 -> 2
- net /USER_BUTTON: track 0.00 -> 74.7 mm, vias 0 -> 2
- net /UART1_TXD: track 0.00 -> 55.5 mm, vias 0 -> 1
- net VBAT: track 0.00 -> 53.7 mm, vias 0 -> 4
- net /I2C0_SDA: track 0.00 -> 53.1 mm, vias 0 -> 2
- net /I2C0_SCL: track 0.00 -> 52.4 mm, vias 0 -> 2
- net /UART1_RXD: track 0.00 -> 50.0 mm, vias 0 -> 1
- net /UART0_RXD: track 0.00 -> 47.4 mm, vias 0 -> 1
- net /PAIR_LED: track 0.00 -> 45.1 mm, vias 0 -> 2
- net /UART0_TXD: track 0.00 -> 39.0 mm, vias 0 -> 1
- net /USER_WS2812: track 0.00 -> 36.6 mm, vias 0 -> 2
- net /EN: track 0.00 -> 35.7 mm, vias 0 -> 2
- net /BKT_IO40: track 0.00 -> 34.1 mm, vias 0 -> 1
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- added copper zone on B.Cu, net GND
- added copper zone on F.Cu, net GND
- added copper zone on In1.Cu, net GND
- added copper zone on In2.Cu, net GND
- added copper zone on F.Cu, net Net-(J15-Pin_2)
- added copper zone on F.Cu, net Net-(JP1-A)
- added copper zone on F.Cu, net Net-(U6-SW)
- added copper zone on In1.Cu, net Net-(U6-SW)
Other:
- board outline added: 97.8 x 50.5 mm
- copper layers 2 -> 4
- board text added: "HB"
- board text added: "I2C0"
- board text added: "ON/OFF"
- board text added: "PWR_3v3"
- board text added: "PWR_in"
- board text added: "PWR_prot"
- board text added: "PlugnPair"
- board text added: "UART"
- board text added: "UserBtn"

Commit message: Done?
Parts:
- added kibuzzard-67CD1FB0: G***, kibuzzard-67CD1FB0, B.Cu at (104.2, 60.6)
- added kibuzzard-67CD1FBD: G***, kibuzzard-67CD1FBD, B.Cu at (107.2, 64.7)
- added kibuzzard-67CD2000: G***, kibuzzard-67CD2000, B.Cu at (119.7, 97.7)
- added kibuzzard-67CD201A: G***, kibuzzard-67CD201A, B.Cu at (158.2, 65.2)
- added kibuzzard-67CD2025: G***, kibuzzard-67CD2025, B.Cu at (134.2, 65.7)
- added kibuzzard-67CD2035: G***, kibuzzard-67CD2035, B.Cu at (114.7, 83.2)
- moved TP3 59.3 mm to (120.7, 65.8)
- moved SW1 59.1 mm to (79.3, 67.3)
- moved TP6 59.0 mm to (95.6, 57.8)
- moved C8 58.9 mm to (152.1, 102.0)
- moved D7 58.9 mm to (149.8, 83.8)
- moved J13 58.9 mm to (142.6, 60.6)
- moved J6 58.9 mm to (162.6, 62.7)
- moved J7 58.9 mm to (162.6, 72.2)
- moved R1 58.9 mm to (167.1, 67.1)
- moved R20 58.9 mm to (152.1, 100.8)
- moved R22 58.9 mm to (150.1, 88.7)
- moved R28 58.9 mm to (165.1, 92.5)
- moved U7 58.9 mm to (135.7, 96.7)
- moved C9 58.9 mm to (114.6, 74.9)
- moved D9 58.9 mm to (156.2, 90.4)
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Routing:
- net GND: track 27.9 -> 49.1 mm, vias 19 -> 74
- net +3V3: track 139.6 -> 159.9 mm
- net /EN: track 35.7 -> 44.1 mm, vias 2 -> 4
- net Net-(JP4-A): track 7.39 -> 10.7 mm
- net Net-(D7-A): track 0.00 -> 2.19 mm
- net VBAT: track 53.7 -> 55.8 mm, vias 4 -> 5
- net Net-(JP1-A): track 29.3 -> 27.7 mm
- net Net-(D5-A): track 0.00 -> 1.43 mm
- net /Servo_Sig_3: track 26.5 -> 27.6 mm
- net +5V: track 103.3 -> 102.3 mm
- net /UART1_RXD: track 50.0 -> 49.0 mm
- net /UART0_TXD: track 39.0 -> 39.8 mm
- net /UART0_RXD: track 47.4 -> 48.2 mm
- net /BKT_IO41: track 31.9 -> 31.3 mm
- net Net-(J2-Pin_3): track 12.7 -> 13.3 mm
- added copper zone on In2.Cu, net Net-(U6-SW)
Other:
- board size 97.8 x 50.5 mm -> 97.7 x 56.8 mm
- board text added: "+"
- board text added: "-"
- board text added: "24v max"
- board text added: "Breakout"
- board text added: "Prog"
